Commit message: Updated ros

File: ros_ws/guboros/urdf/pad_cell.urdf (robot description, URDF)
Before this commit: robot crx20ia_l, 22 links, 21 joints
Links:
- link J1_link: geometry collision mesh filename=package://guboros/urdf/meshes/crx20ia_l/collision/j1.stl scale=0.001 0.001 0.001; visual mesh filename=package://guboros/urdf/meshes/crx20ia_l/visual/j1.stl scale=0.001 0.001 0.001
- link J2_link: geometry collision mesh filename=package://guboros/urdf/meshes/crx20ia_l/collision/j2.stl scale=0.001 0.001 0.001; visual mesh filename=package://guboros/urdf/meshes/crx20ia_l/visual/j2.stl scale=0.001 0.001 0.001
- link J3_link: geometry collision mesh filename=package://guboros/urdf/meshes/crx20ia_l/collision/j3.stl scale=0.001 0.001 0.001; visual mesh filename=package://guboros/urdf/meshes/crx20ia_l/visual/j3.stl scale=0.001 0.001 0.001
- link J4_link: geometry collision mesh filename=package://guboros/urdf/meshes/crx20ia_l/collision/j4.stl scale=0.001 0.001 0.001; visual mesh filename=package://guboros/urdf/meshes/crx20ia_l/visual/j4.stl scale=0.001 0.001 0.001
- link J5_link: geometry collision mesh filename=package://guboros/urdf/meshes/crx20ia_l/collision/j5.stl scale=0.001 0.001 0.001; visual mesh filename=package://guboros/urdf/meshes/crx20ia_l/visual/j5.stl scale=0.001 0.001 0.001
- link J6_link: geometry collision mesh filename=package://guboros/urdf/meshes/crx20ia_l/collision/j6.stl scale=0.001 0.001 0.001; visual mesh filename=package://guboros/urdf/meshes/crx20ia_l/visual/j6.stl scale=0.001 0.001 0.001
- link base_link: geometry collision mesh filename=package://guboros/urdf/meshes/crx20ia_l/collision/base.stl scale=0.001 0.001 0.001; visual mesh filename=package://guboros/urdf/meshes/crx20ia_l/visual/base.stl scale=0.001 0.001 0.001
- link t1table: geometry collision box size=.76 1.02 .94; visual mesh filename=package://guboros/urdf/meshes/others/visual/table.stl
