Commit message: gian finer

File: ros_ws/finger_pkg/urdf/finger.urdf (robot description, URDF)
Before this commit: robot two_segment_arm, 3 links, 2 joints
Links:
- link link2: geometry collision mesh filename=package://finger_pkg/urdf/meshes/finger/visual/Joint.stl scale=0.001 0.001 0.001; visual mesh filename=package://finger_pkg/urdf/meshes/finger/visual/Joint.stl scale=0.001 0.001 0.001
